Commit message: Ackerman robot now has the four wheels in Gazebo. Added steering wheel inertia

File: delta_description/diffdrive_urdf/ackerman_robot.urdf.xacro (robot description, xacro)
@@ -60,6 +60,42 @@
         </collision>
     </link>
-    <link name="steering_FR_link"/>
-    <link name="steering_FL_link"/>
+    <link name="steering_FR_link">
+        <visual>
+            <geometry>
+                <box size="0.01 0.01 0.01"/>
+            </geometry>
+            <origin xyz="0 0 0" rpy="0 0 0"/>
+        </visual>
+        <inertial>
+            <mass value="0.1"/>
+            <origin xyz="0 0 0" rpy="0 0 0"/>
+            <inertia ixx="0.01" ixy="0" ixz="0" iyy="0.01" iyz="0" izz="0.01"/>
+        </inertial>
+        <collision>
+            <geometry>
+                <box size="0.01 0.01 0.01"/>
+            </geometry>
+            <origin xyz="0 0 0" rpy="0 0 0"/>
+        </collision>
+    </link>
+    <link name="steering_FL_link">
+        <visual>
+            <geometry>
+                <box size="0.01 0.01 0.01"/>
+            </geometry>
+            <origin xyz="0 0 0" rpy="0 0 0"/>
+        </visual>
+        <inertial>
+            <mass value="0.1"/>
+            <origin xyz="0 0 0" rpy="0 0 0"/>
+            <inertia ixx="0.01" ixy="0" ixz="0" iyy="0.01" iyz="0" izz="0.01"/>
+        </inertial>
+        <collision>
+            <geometry>
+                <box size="0.01 0.01 0.01"/>
+            </geometry>
+            <origin xyz="0 0 0" rpy="0 0 0"/>
+        </collision>
+    </link>
     <joint name="chassis_wheel_RR_joint" type="continuous">
         <parent link="chassis_link"/>
@@ -72,5 +108,5 @@
     <joint name="chassis_wheel_RL_joint" type="continuous">
         <parent link="chassis_link"/>
-        <child link="rwheel_link2"/>ackerman_robot.urdf
+        <child link="rwheel_link2"/>
         <origin xyz="-${off_x} ${off_y} -${off_z} " rpy="0 0 0"/>
         <axis xyz="0 1 0"/> <!-- eje de rotación del joint, se define en coordenadas del link padre -->

Commit message: Adjust joystick priority in twist_mux.yaml and refine URDF properties for ackerman_robot; update control_gap_ttc.py to remove steering limits and enhance TTC break logic in ttc_break_node.py; modify wall distance parameter in dist_finder.py

File: delta_description/diffdrive_urdf/ackerman_robot.urdf.xacro (robot description, xacro)
@@ -1,13 +1,13 @@
 <?xml version='1.0'?>
 <robot xmlns:xacro="http://www.ros.org/wiki/xacro" name="ackerman_robot">
-    <xacro:property name="lx_box" value="${41/10}" /><!-- se aconseja definir porpiedades gemetricas con estas lineas -->
-    <xacro:property name="ly_box" value="${16/10}" />
-    <xacro:property name="lz_box" value="${13.3/10}" />
-    <xacro:property name="off_x" value="${12.55/10}" />
-    <xacro:property name="off_z" value="${5.45/10}" />
-    <xacro:property name="off_z_chasi" value="${6.65/10}" />
-    <xacro:property name="rad_cil" value="${10.2/2/10}" />
-    <xacro:property name="altura" value="${4.5/10}" />
-    <xacro:property name="off_y" value="${12.15/10}" />
+    <xacro:property name="lx_box" value="${41/100}" /><!-- se aconseja definir porpiedades gemetricas con estas lineas -->
+    <xacro:property name="ly_box" value="${16/100}" />
+    <xacro:property name="lz_box" value="${13.3/100}" />
+    <xacro:property name="off_x" value="${12.55/100}" />
+    <xacro:property name="off_z" value="${5.45/100}" />
+    <xacro:property name="off_z_chasi" value="${6.65/100}" />
+    <xacro:property name="rad_cil" value="${10.2/2/100}" />
+    <xacro:property name="altura" value="${4.5/100}" />
+    <xacro:property name="off_y" value="${12.15/100}" />
   <xacro:macro name="wheel_macro" params="w_name w_radius w_lenght ">
     <link name="${w_name}">  <!-- este link es un cuerpo con unos atributos de visual, inercia y colision -->
